Commit message: re-adds choo_2, completes new agv model, and adds motors.py from og ugv_sim

File: agv_model/untitled_agv/model.urdf.xacro (robot description, xacro)
@@ -4,24 +4,24 @@
     <!-- physical parameters of robot, all in SI (meters, kg) -->
     <!-- base dimensions -->
-    <xacro:property name="base_mass" value="45.36" />
-    <xacro:property name="base_width" value="0.5588" />     <!-- width=y -->
-    <xacro:property name="base_length" value="0.9398" />    <!-- length=x -->
-    <xacro:property name="base_height" value="0.305" />     <!-- height=z -->
+    <xacro:property name="base_mass" value="17.216" />
+    <xacro:property name="base_width" value="0.78" />     <!-- width=y -->
+    <xacro:property name="base_length" value="0.92" />    <!-- length=x -->
+    <xacro:property name="base_height" value="0.5" />     <!-- height=z -->
     <!-- wheel properties -->
-    <xacro:property name="wheel_radius" value="0.10795" />
-    <xacro:property name="wheel_width" value="0.059" />
+    <xacro:property name="wheel_radius" value="0.1016" />
+    <xacro:property name="wheel_width" value=".0635" />
     <!-- differential properties -->
-    <xacro:property name="wheel_mass" value="1.179" />
-    <xacro:property name="wheelbase" value="0.67" />
-    <xacro:property name="track_width" value="0.67" />
-    <xacro:property name="wheel_offset_x" value="${wheelbase / 2}" />
-    <xacro:property name="wheel_offset_y" value="${track_width / 2}" />
-    <xacro:property name="wheel_offset_z" value="-0.186475" />
+    <xacro:property name="wheel_mass" value="1.179" />      <!--need-->
+    <xacro:property name="wheelbase" value=".0725" />       <!--need-->
+    <xacro:property name="track_width" value=".5445" />
+    <xacro:property name="wheel_offset_x" value="${wheelbase / 2}" />    <!--length=x-->
+    <xacro:property name="wheel_offset_y" value="${(base_width / 2) + (wheel_width/2)}" />  <!--width=y-->
+    <xacro:property name="wheel_offset_z" value="${(base_height / 2)}" />          <!--height=z-->     <!--need-->
     <!-- lidar stalk properties -->
-    <xacro:property name="lidar_stalk_height" value="0.330" />
+    <xacro:property name="lidar_stalk_height" value="0.430" />
     <xacro:property name="lidar_stalk_side" value="0.020" />
-    <xacro:property name="lidar_stalk_offset_x" value="-0.1311" />
-    <xacro:property name="lidar_stalk_offset_y" value="0.0" />
-    <xacro:property name="lidar_stalk_offset_z" value="${base_height / 2}" />
+    <xacro:property name="lidar_stalk_offset_x" value="-0.1311" />         <!--need-->
+    <xacro:property name="lidar_stalk_offset_y" value="0.0" />              <!--need-->
+    <xacro:property name="lidar_stalk_offset_z" value="${base_height / 2}" />      <!--need-->
     <!-- lidar properties -->
     <xacro:property name="lidar_mass" value="0.830" />
@@ -40,9 +40,13 @@
     <xacro:property name="cam_offset_y" value="0.0" />
     <xacro:property name="cam_offset_z" value="${(base_height / 2) + cam_height}" />
+    <!-- caster properties -->
+    <xacro:property name="caster_offset_x" value="0.3857 " />
+    <xacro:property name="caster_offset_y" value="0.1756" />
+    <xacro:property name="caster_offset_z" value="${(base_height / 2)}" />     <!--${(base_height / 2) + cam_height}-->
     <!--
         Include other xacro files for simulation plugins, Gazebo references, and macros
     -->
-    <xacro:include filename="$(find ugv_description)/urdf/choo_2/model.gazebo" />
-    <xacro:include filename="$(find ugv_description)/urdf/choo_2/model.macro" />
+    <xacro:include filename="$(find agv_model)/choo_2/model.gazebo" />
+    <xacro:include filename="$(find agv_model)/choo_2/model.macro" />
     <!--
         objects contained within the gazebo tags are for Gazebo simulation use only, ignored otherwise.
@@ -57,19 +61,16 @@
     <xacro:wheel name="front_left_wheel" wheel_radius="${wheel_radius}" wheel_width="${wheel_width}" wheel_mass="${wheel_mass}"/>
     <xacro:wheel_joint name="front_left_wheel" x_offset="${wheel_offset_x}" y_offset="${wheel_offset_y}" z_offset="${wheel_offset_z}" reflect_x="1" reflect_y="1"/>
-    <!-- back left wheel -->
-    <!-- <xacro:wheel name="back_left_wheel" wheel_radius="${wheel_radius}" wheel_width="${wheel_width}" wheel_mass="${wheel_mass}"/>
-    <xacro:wheel_joint name="back_left_wheel" x_offset="${wheel_offset_x}" y_offset="${wheel_offset_y}" z_offset="${wheel_offset_z}" reflect_x="-1" reflect_y="1"/> -->
     <!-- front right wheel -->
     <xacro:wheel name="front_right_wheel" wheel_radius="${wheel_radius}" wheel_width="${wheel_width}" wheel_mass="${wheel_mass}"/>
     <xacro:wheel_joint name="front_right_wheel" x_offset="${wheel_offset_x}" y_offset="${wheel_offset_y}" z_offset="${wheel_offset_z}" reflect_x="1" reflect_y="-1"/>
-    <!-- back right wheel-->
-    <!-- <xacro:wheel name="back_right_wheel" wheel_radius="${wheel_radius}" wheel_width="${wheel_width}" wheel_mass="${wheel_mass}"/>
-    <xacro:wheel_joint name="back_right_wheel" x_offset="${wheel_offset_x}" y_offset="${wheel_offset_y}" z_offset="${wheel_offset_z}" reflect_x="-1" reflect_y="-1"/> -->
     <!-- back left caster -->
-    <xacro:caster_total name="back_left_caster" radius="0.294425" mass="5" />
-    <xacro:caster_joint name="back_left_caster" x_offset="${wheel_offset_x}" y_offset="0" z_offset="0" reflect_x="-1" reflect_y="1"/>
+    <xacro:caster_total name="back_left_caster" radius="${wheel_radius*0.95}" mass="${wheel_mass}" />
+    <xacro:caster_joint name="back_left_caster" x_offset="${caster_offset_x}" y_offset="${caster_offset_y}" z_offset="${caster_offset_z}" reflect_x="-1" reflect_y="1"/>
     <!-- back right caster -->
-    <!-- <xacro:caster_total name="back_right_caster" radius="${wheel_radius}" mass="${wheel_mass}" />
-    <xacro:caster_joint name="back_right_caster" x_offset="${wheel_offset_x}" y_offset="${wheel_offset_y / 2}" z_offset="${wheel_offset_z}" reflect_x="-1" reflect_y="-1"/> -->
+    <xacro:caster_total name="back_right_caster" radius="${wheel_radius*0.95}" mass="${wheel_mass}" />
+    <xacro:caster_joint name="back_right_caster" x_offset="${caster_offset_x}" y_offset="${caster_offset_y}" z_offset="${caster_offset_z}" reflect_x="-1" reflect_y="-1"/> -->
+    <!--front caster wheel-->
+    <xacro:caster_total name="front_caster" radius="${wheel_radius*0.95}" mass="${wheel_mass}" />
+    <xacro:caster_joint name="front_caster" x_offset="0.311" y_offset="0" z_offset="${caster_offset_z}" reflect_x="1" reflect_y="1"/>
     <!-- lidar stalk -->
     <xacro:box_total name="lidar_stalk" mass="0.14982" width="${lidar_stalk_side}" length="${lidar_stalk_side}" height="${lidar_stalk_height}" />
@@ -82,5 +83,5 @@
     </joint>
     <!-- lidar link -->
-    <link name="velodyne">
+    <link name="velodyne">0.3857
         <gazebo reference="velodyne">
         </gazebo>
